File: Kicad/Project SBO Schism/board.kicad_pcb (KiCad board)
At the start: 2 copper layers, 122.3 x 118.1 mm, 50 parts

Commit message: the beginning of the wiring
must be neat must be neat must be neat must be neat must be neat must be neat
Routing:
- net col_pinky: track 13.3 -> 141.7 mm, vias 0 -> 1
- net P0: track 25.2 -> 70.3 mm
- net VCC: track 20.4 -> 63.7 mm
- net RST: track 13.3 -> 49.0 mm
- net pinky_extra: track 0.00 -> 30.6 mm
- net pinky_bottom: track 0.00 -> 29.9 mm
- net pinky_top: track 0.00 -> 29.7 mm
- net pinky_home: track 0.00 -> 29.7 mm
- net GND: track 38.4 -> 55.7 mm
- net row_top: track 18.3 -> 22.6 mm
- net row_home: track 18.3 -> 22.6 mm
- net row_extra: track 18.3 -> 22.6 mm
- net row_bottom: track 18.3 -> 22.6 mm

Commit message: Work continues
Routing:
- net row_bottom: track 22.6 -> 130.6 mm
- net row_extra: track 22.6 -> 129.9 mm
- net row_home: track 22.6 -> 126.9 mm
- net row_top: track 22.6 -> 124.8 mm
- net ring_extra: track 0.00 -> 31.2 mm
- net ring_top: track 0.00 -> 30.9 mm
- net middle_home: track 0.00 -> 4.32 mm
- net middle_extra: track 0.00 -> 4.32 mm
- net middle_bottom: track 0.00 -> 4.32 mm
- net index_top: track 0.00 -> 4.32 mm
- net index_home: track 0.00 -> 4.32 mm
- net index_extra: track 0.00 -> 4.32 mm
- net index_bottom: track 0.00 -> 4.32 mm
- net ring_home: track 0.00 -> 4.32 mm
- net ring_bottom: track 0.00 -> 4.32 mm
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